Commit message: Add robot descriptions

File: whole_body/urdf/g1_29dof.urdf (robot description, URDF)
Before this commit: robot g1_23dof_rev_1_0, 48 links, 47 joints
Links:
- removed link left_wrist_roll_rubber_hand
- removed link right_wrist_roll_rubber_hand
- added link left_rubber_hand, mass 0.170; visual mesh filename=meshes/left_rubber_hand.STL
- added link left_wrist_pitch_link, mass 0.48404956; collision mesh filename=meshes/left_wrist_pitch_link.STL; visual mesh filename=meshes/left_wrist_pitch_link.STL
- added link left_wrist_roll_link, mass 0.08544498; collision mesh filename=meshes/left_wrist_roll_link.STL; visual mesh filename=meshes/left_wrist_roll_link.STL
- added link left_wrist_yaw_link, mass 0.08457647; collision mesh filename=meshes/left_wrist_yaw_link.STL; visual mesh filename=meshes/left_wrist_yaw_link.STL
- added link right_rubber_hand, mass 0.170; visual mesh filename=meshes/right_rubber_hand.STL
- added link right_wrist_pitch_link, mass 0.48404956; collision mesh filename=meshes/right_wrist_pitch_link.STL; visual mesh filename=meshes/right_wrist_pitch_link.STL
- added link right_wrist_roll_link, mass 0.08544498; collision mesh filename=meshes/right_wrist_roll_link.STL; visual mesh filename=meshes/right_wrist_roll_link.STL
- added link right_wrist_yaw_link, mass 0.08457647; collision mesh filename=meshes/right_wrist_yaw_link.STL; visual mesh filename=meshes/right_wrist_yaw_link.STL
- added link waist_roll_link, mass 0.086; visual mesh filename=meshes/waist_roll_link_rev_1_0.STL
- added link waist_yaw_link, mass 0.214; visual mesh filename=meshes/waist_yaw_link_rev_1_0.STL
- link head_link: geometry collision mesh filename=meshes/head_link.STL; visual mesh filename=meshes/head_link.STL
- link left_ankle_pitch_link: geometry collision mesh filename=meshes/left_ankle_pitch_link.STL; visual mesh filename=meshes/left_ankle_pitch_link.STL
- link left_ankle_roll_link: geometry collision sphere radius=0.005; collision sphere radius=0.005
- link left_elbow_link: geometry collision mesh filename=meshes/left_elbow_link.STL; visual mesh filename=meshes/left_elbow_link.STL
- link left_hip_pitch_link: geometry collision mesh filename=meshes/left_hip_pitch_link.STL; visual mesh filename=meshes/left_hip_pitch_link.STL
- link left_hip_roll_link: geometry collision mesh filename=meshes/left_hip_roll_link.STL; visual mesh filename=meshes/left_hip_roll_link.STL
- link left_hip_yaw_link: geometry collision mesh filename=meshes/left_hip_yaw_link.STL; visual mesh filename=meshes/left_hip_yaw_link.STL
- link left_knee_link: geometry collision mesh filename=meshes/left_knee_link.STL; visual mesh filename=meshes/left_knee_link.STL
- link left_shoulder_pitch_link: geometry collision cylinder length=0.05 radius=0.03; visual mesh filename=meshes/left_shoulder_pitch_link.STL
- link left_shoulder_roll_link: geometry collision cylinder length=0.03 radius=0.03; visual mesh filename=meshes/left_shoulder_roll_link.STL
- link left_shoulder_yaw_link: geometry collision mesh filename=meshes/left_shoulder_yaw_link.STL; visual mesh filename=meshes/left_shoulder_yaw_link.STL
- link logo_link: geometry collision mesh filename=meshes/logo_link.STL; visual mesh filename=meshes/logo_link.STL
- link pelvis: geometry visual mesh filename=meshes/pelvis.STL
- link pelvis_contour_link: geometry collision mesh filename=meshes/pelvis_contour_link.STL; visual mesh filename=meshes/pelvis_contour_link.STL
- link right_ankle_pitch_link: geometry collision mesh filename=meshes/right_ankle_pitch_link.STL; visual mesh filename=meshes/right_ankle_pitch_link.STL
- link right_ankle_roll_link: geometry collision sphere radius=0.005; collision sphere radius=0.005
- link right_elbow_link: geometry collision mesh filename=meshes/right_elbow_link.STL; visual mesh filename=meshes/right_elbow_link.STL
- link right_hip_pitch_link: geometry collision mesh filename=meshes/right_hip_pitch_link.STL; visual mesh filename=meshes/right_hip_pitch_link.STL
- link right_hip_roll_link: geometry collision mesh filename=meshes/right_hip_roll_link.STL; visual mesh filename=meshes/right_hip_roll_link.STL
- link right_hip_yaw_link: geometry collision mesh filename=meshes/right_hip_yaw_link.STL; visual mesh filename=meshes/right_hip_yaw_link.STL
- link right_knee_link: geometry collision mesh filename=meshes/right_knee_link.STL; visual mesh filename=meshes/right_knee_link.STL
- link right_shoulder_pitch_link: geometry collision cylinder length=0.05 radius=0.03; visual mesh filename=meshes/right_shoulder_pitch_link.STL
- link right_shoulder_roll_link: geometry collision cylinder length=0.03 radius=0.03; visual mesh filename=meshes/right_shoulder_roll_link.STL
- link right_shoulder_yaw_link: geometry collision mesh filename=meshes/right_shoulder_yaw_link.STL; visual mesh filename=meshes/right_shoulder_yaw_link.STL
- link torso_link: geometry collision mesh filename=meshes/torso_link_rev_1_0.STL; visual mesh filename=meshes/torso_link_rev_1_0.STL
Joints:
- added joint left_hand_palm_joint: type fixed, parent left_wrist_yaw_link, child left_rubber_hand, origin xyz=0.0415 0.003 0 rpy=0 0 0
- added joint left_wrist_pitch_joint: type revolute, parent left_wrist_roll_link, child left_wrist_pitch_link, origin xyz=0.038 0 0 rpy=0 0 0, axis 0 1 0, limit lower=-1.614429558 upper=1.614429558 effort=5 velocity=22
- added joint left_wrist_yaw_joint: type revolute, parent left_wrist_pitch_link, child left_wrist_yaw_link, origin xyz=0.046 0 0 rpy=0 0 0, axis 0 0 1, limit lower=-1.614429558 upper=1.614429558 effort=5 velocity=22
- added joint right_hand_palm_joint: type fixed, parent right_wrist_yaw_link, child right_rubber_hand, origin xyz=0.0415 -0.003 0 rpy=0 0 0
- added joint right_wrist_pitch_joint: type revolute, parent right_wrist_roll_link, child right_wrist_pitch_link, origin xyz=0.038 0 0 rpy=0 0 0, axis 0 1 0, limit lower=-1.614429558 upper=1.614429558 effort=5 velocity=22
- added joint right_wrist_yaw_joint: type revolute, parent right_wrist_pitch_link, child right_wrist_yaw_link, origin xyz=0.046 0 0 rpy=0 0 0, axis 0 0 1, limit lower=-1.614429558 upper=1.614429558 effort=5 velocity=22
- added joint waist_pitch_joint: type revolute, parent waist_roll_link, child torso_link, origin xyz=0 0 0 rpy=0 0 0, axis 0 1 0, limit lower=-0.52 upper=0.52 effort=50 velocity=37
- added joint waist_roll_joint: type revolute, parent waist_yaw_link, child waist_roll_link, origin xyz=-0.0039635 0 0.044 rpy=0 0 0, axis 1 0 0, limit lower=-0.52 upper=0.52 effort=50 velocity=37
- joint left_hand_point_contact_fix_joint: origin xyz=0.17 0.0 0.0 rpy=0 0 0 -> xyz=0.05 0.0 0.0 rpy=0 0 0; parent left_wrist_roll_rubber_hand -> left_rubber_hand
- joint left_wrist_roll_joint: child left_wrist_roll_rubber_hand -> left_wrist_roll_link
- joint right_hand_point_contact_fix_joint: origin xyz=0.17 0.0 0.0 rpy=0 0 0 -> xyz=0.05 0.0 0.0 rpy=0 0 0; parent right_wrist_roll_rubber_hand -> right_rubber_hand
- joint right_wrist_roll_joint: child right_wrist_roll_rubber_hand -> right_wrist_roll_link
- joint waist_yaw_joint: child torso_link -> waist_yaw_link; origin xyz=-0.0039635 0 0.044 rpy=0 0 0 -> xyz=0 0 0 rpy=0 0 0
